File: LSN50/v1.3/LoRa ST Sensor Node v1.3.brd (EAGLE design)
At the start: 58 x 43.5 mm, 49 parts, among them Q8 BSS138-7-F, SW1 MSS22D-18G2-2P2T-H2MM, T1 PMOS, U1 NGFF_M2_KEY_E_SHIELD, U2 RT9266

Commit message: typo , fix
Parts:
- R14: value 10K -> 10M
Changed lines of the file:
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@@
 <attribute name="VALUE" x="-5.24" y="-6.833" size="0.8128" layer="27" rot="R270"/>
 </element>
-<element name="R14" library="dragino" package="R0603" value="10K" x="-2.794" y="-6.096" smashed="yes">
+<element name="R14" library="dragino" package="R0603" value="10M" x="-2.794" y="-6.096" smashed="yes">
 <attribute name="NAME" x="-7.239" y="-6.223" size="0.8128" layer="25" font="vector"/>
 <attribute name="VALUE" x="-4.699" y="-7.493" size="0.8128" layer="27"/>
