File: LSN50/v1.3/LoRa ST Sensor Node v1.3.sch (EAGLE design)
At the start: 47 parts, among them Q8 BSS138-7-F, SW1 MSS22D-18G2-2P2T-H2MM, T1 PMOS, U1 NGFF_M2_KEY_E_SHIELD, U2 RT9266

Commit message: typo , fix
Parts:
- R14: value 10K -> 10M
Changed lines of the file:
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@@
 <part name="R12" library="dragino" deviceset="R-US_" device="R0603" value="10K"/>
 <part name="R13" library="dragino" deviceset="R-US_" device="R0603" value="0Ω"/>
-<part name="R14" library="dragino" deviceset="R-US_" device="R0603" value="10K"/>
+<part name="R14" library="dragino" deviceset="R-US_" device="R0603" value="10M"/>
 <part name="GND4" library="supply1" deviceset="GND" device=""/>
 <part name="C1" library="dragino" deviceset="C-EU" device="C0603" value="100pF 10V"/>
